File: Overview & Details/Protoboard/Protoboard_Activity/Project_1-USB_C/Activity_1.kicad_pcb (KiCad board)
At the start: 2 copper layers, 0 parts

Commit message: Activity 1
Parts:
- added H1: MountingHole, MountingHole:MountingHole_2.5mm, F.Cu at (25.0, 65.0)
- added H2: MountingHole, MountingHole:MountingHole_2.5mm, F.Cu at (25.0, 115.0)
- added H3: MountingHole, MountingHole:MountingHole_2.5mm, F.Cu at (95.0, 65.0)
- added H4: MountingHole, MountingHole:MountingHole_2.5mm, F.Cu at (95.0, 115.0)
- added J1: USB_C, Project_1-USB_C:USB_C_Receptacle_XKB_U262-161N-4BVC11, F.Cu at (27.0, 90.0)
- added Je: Conn_01x04, Connector_PinHeader_2.54mm:PinHeader_1x04_P2.54mm_Vertical, F.Cu at (24.0, 80.0)
Routing:
- net (no net): track 0.00 -> 243.8 mm, vias 0 -> 508
- net Net-(J1-PadA1): track 0.00 -> 54.4 mm
- net /+5: track 0.00 -> 26.4 mm
Other:
- board outline added: 80 x 60 mm
