File: Overview & Details/LEDboard/LEDboard_Activity/LED_Board_s_.sch (KiCad schematic (older format))
At the start: 6 parts, among them J1 Conn_01x04

Commit message: project1
Parts:
- added D10, D11, D12, D13, D14, D15, D16, D17, D18, D19, D2, D20, D21, D22, D23, D24, D25, D26, D27, D28, D29, D3, D30, D31, D32, D33, D34, D35, D36, D37, D38, D39, D4, D40, D41, D42, D43, D44, D45, D46, D47, D48, D5, D6, D7, D8, D9: APA102-2020, LED_SMD:LED-APA102-2020, symbol LED:APA102-2020
- added FID1, FID2: Fiducial, Fiducial:Fiducial_0.5mm_Mask1mm, symbol Mechanical:Fiducial
Connections:
- wire segments 9 -> 125
Other:
- note added: "n/c\n"
- note removed: "n/c"
