File: Overview & Details/LEDboard/LEDboard_Activity/LED_Board_s_.kicad_pcb (KiCad board)
At the start: 2 copper layers, 0 parts

Commit message: project1
Parts:
- added D1: APA102-2020, LED_SMD:LED-APA102-2020, F.Cu at (28.6, 25.8)
- added D10: APA102-2020, LED_SMD:LED-APA102-2020, F.Cu at (63.5, 35.3)
- added D11: APA102-2020, LED_SMD:LED-APA102-2020, F.Cu at (46.0, 35.3)
- added D12: APA102-2020, LED_SMD:LED-APA102-2020, F.Cu at (28.6, 35.3)
- added D13: APA102-2020, LED_SMD:LED-APA102-2020, F.Cu at (28.6, 44.8)
- added D14: APA102-2020, LED_SMD:LED-APA102-2020, F.Cu at (46.0, 44.8)
- added D15: APA102-2020, LED_SMD:LED-APA102-2020, F.Cu at (63.5, 44.8)
- added D16: APA102-2020, LED_SMD:LED-APA102-2020, F.Cu at (80.9, 44.8)
- added D17: APA102-2020, LED_SMD:LED-APA102-2020, F.Cu at (98.4, 44.8)
- added D18: APA102-2020, LED_SMD:LED-APA102-2020, F.Cu at (115.9, 44.8)
- added D19: APA102-2020, LED_SMD:LED-APA102-2020, F.Cu at (115.9, 54.3)
- added D2: APA102-2020, LED_SMD:LED-APA102-2020, F.Cu at (46.0, 25.8)
- added D20: APA102-2020, LED_SMD:LED-APA102-2020, F.Cu at (98.4, 54.3)
- added D21: APA102-2020, LED_SMD:LED-APA102-2020, F.Cu at (80.9, 54.3)
- added D22: APA102-2020, LED_SMD:LED-APA102-2020, F.Cu at (63.5, 54.3)
- added D23: APA102-2020, LED_SMD:LED-APA102-2020, F.Cu at (46.0, 54.3)
- added D24: APA102-2020, LED_SMD:LED-APA102-2020, F.Cu at (28.6, 54.3)
- added D25: APA102-2020, LED_SMD:LED-APA102-2020, F.Cu at (28.6, 63.9)
- added D26: APA102-2020, LED_SMD:LED-APA102-2020, F.Cu at (46.0, 63.9)
- added D27: APA102-2020, LED_SMD:LED-APA102-2020, F.Cu at (63.5, 63.9)
- added D28: APA102-2020, LED_SMD:LED-APA102-2020, F.Cu at (80.9, 63.9)
- added D29: APA102-2020, LED_SMD:LED-APA102-2020, F.Cu at (98.4, 63.9)
- added D3: APA102-2020, LED_SMD:LED-APA102-2020, F.Cu at (63.5, 25.8)
- added D30: APA102-2020, LED_SMD:LED-APA102-2020, F.Cu at (115.9, 63.9)
- added D31: APA102-2020, LED_SMD:LED-APA102-2020, F.Cu at (115.9, 73.4)
- added D32: APA102-2020, LED_SMD:LED-APA102-2020, F.Cu at (98.4, 73.4)
- added D33: APA102-2020, LED_SMD:LED-APA102-2020, F.Cu at (80.9, 73.4)
- added D34: APA102-2020, LED_SMD:LED-APA102-2020, F.Cu at (63.5, 73.4)
- added D35: APA102-2020, LED_SMD:LED-APA102-2020, F.Cu at (46.0, 73.4)
- added D36: APA102-2020, LED_SMD:LED-APA102-2020, F.Cu at (28.6, 73.4)
- added D37: APA102-2020, LED_SMD:LED-APA102-2020, F.Cu at (28.6, 82.9)
- added D38: APA102-2020, LED_SMD:LED-APA102-2020, F.Cu at (46.0, 82.9)
- added D39: APA102-2020, LED_SMD:LED-APA102-2020, F.Cu at (63.5, 82.9)
- added D4: APA102-2020, LED_SMD:LED-APA102-2020, F.Cu at (80.9, 25.8)
- added D40: APA102-2020, LED_SMD:LED-APA102-2020, F.Cu at (80.9, 82.9)
- added D41: APA102-2020, LED_SMD:LED-APA102-2020, F.Cu at (98.4, 82.9)
- added D42: APA102-2020, LED_SMD:LED-APA102-2020, F.Cu at (115.9, 82.9)
- added D43: APA102-2020, LED_SMD:LED-APA102-2020, F.Cu at (115.9, 92.4)
- added D44: APA102-2020, LED_SMD:LED-APA102-2020, F.Cu at (98.4, 92.4)
- added D45: APA102-2020, LED_SMD:LED-APA102-2020, F.Cu at (80.9, 92.4)
- added D46: APA102-2020, LED_SMD:LED-APA102-2020, F.Cu at (63.5, 92.4)
- added D47: APA102-2020, LED_SMD:LED-APA102-2020, F.Cu at (46.0, 92.4)
- added D48: APA102-2020, LED_SMD:LED-APA102-2020, F.Cu at (28.6, 92.4)
- added D5: APA102-2020, LED_SMD:LED-APA102-2020, F.Cu at (98.4, 25.8)
- added D6: APA102-2020, LED_SMD:LED-APA102-2020, F.Cu at (115.9, 25.8)
- added D7: APA102-2020, LED_SMD:LED-APA102-2020, F.Cu at (115.9, 35.3)
- added D8: APA102-2020, LED_SMD:LED-APA102-2020, F.Cu at (98.4, 35.3)
- added D9: APA102-2020, LED_SMD:LED-APA102-2020, F.Cu at (80.9, 35.3)
- added FID1: Fiducial, Fiducial:Fiducial_0.5mm_Mask1mm, F.Cu at (18.2, 33.9)
- added FID2: Fiducial, Fiducial:Fiducial_0.5mm_Mask1mm, F.Cu at (124.4, 84.0)
- added H1: MountingHole, MountingHole:MountingHole_3.5mm_Pad, F.Cu at (20.0, 25.9)
- added H2: MountingHole_Pad, MountingHole:MountingHole_3.5mm_Pad_Via, F.Cu at (20.0, 92.3)
- added H3: MountingHole, MountingHole:MountingHole_3.5mm_Pad, F.Cu at (124.5, 25.9)
- added H4: MountingHole, MountingHole:MountingHole_3.5mm_Pad, F.Cu at (124.5, 92.3)
- added J1: Conn_01x04, Connector_PinHeader_2.54mm:PinHeader_1x04_P2.54mm_Vertical, B.Cu at (19.9, 64.6)
Routing:
- net GND: track 0.00 -> 246.4 mm, vias 0 -> 271
- net +5VD: track 0.00 -> 212.6 mm
- net /SDI: track 0.00 -> 48.2 mm
- net /CKI: track 0.00 -> 41.9 mm
- net Net-(D7-Pad3): track 0.00 -> 15.8 mm
- net Net-(D7-Pad2): track 0.00 -> 15.8 mm
- net Net-(D5-Pad3): track 0.00 -> 15.8 mm
- net Net-(D5-Pad2): track 0.00 -> 15.8 mm
- net Net-(D46-Pad3): track 0.00 -> 15.8 mm
- net Net-(D46-Pad2): track 0.00 -> 15.8 mm
- net Net-(D45-Pad3): track 0.00 -> 15.8 mm
- net Net-(D45-Pad2): track 0.00 -> 15.8 mm
- net Net-(D43-Pad3): track 0.00 -> 15.8 mm
- net Net-(D43-Pad2): track 0.00 -> 15.8 mm
- net Net-(D41-Pad3): track 0.00 -> 15.8 mm
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- added copper zone on F.Cu, net +5VD
- added copper zone on B.Cu, net GND
- added copper zone on F.Cu, net GND
Other:
- board outline added: 114.3 x 76.2 mm
- net class jlpcb added: clearance 0.127, trace_width 0.25, via_dia 0.8, via_drill 0.4

Commit message: LED board fixes
Routing:
- net GND: track 246.4 -> 350.8 mm, vias 271 -> 270
