File: Overview & Details/Powerboard/Powerboard_Activity/Power_Board.sch (KiCad schematic (older format))
At the start: 29 parts

Commit message: Updates to power boarcd
Parts:
- added C?: 82pF, symbol Device:C
- added C?: 10µF, symbol Device:CP1
- added C?: 1µF, symbol Device:C
- added C?: 47µF, symbol Device:CP1
- added C?: 100µF, symbol Device:CP1
- added C?: 22µF, symbol Device:CP1
- added D?: PMEG2010AEH, Diode_SMD:D_SOD-123F, symbol Diode:PMEG2010AEH
- added L?: 10µH, symbol Device:L
- added L?: 22µH, symbol Device:L
- added R?: 300kΩ, symbol Device:R_Small_US
- added R?: 130kΩ, symbol Device:R_Small_US
- added U?: MAX735CSA-Regulator_Switching, symbol Power_Board:MAX735CSA-Regulator_Switching
Connections:
- net +5VA: now also C?.1, C?.1, U?.1 (~SHDN), U?.8 (V+)
- net -5VA: now also C?.2, L?.2
- net GNDS: now also C?.1, C?.1, C?.2, C?.2, C?.2, C?.2, L?.2, R?.1, U?.6 (GND)
- new net: C?.1, R?.2, U?.2 (Vref)
- new net: R?.1, R?.2, U?.3 (SS)
- new net: C?.1, U?.4 (CC)
- new net: C?.2, D?.2 (A), L?.1, U?.5 (Vout)
- new net: D?.1 (K), L?.1, U?.7 (LX)
